Commit message: URDF loaded successfully in RViz

File: maze_robot_v1_description/urdf/maze_robot_v1.xacro (robot description, xacro)
@@ -146,24 +146,4 @@
 <link name="base_top_1">
   <inertial>
-    <origin rpy="0 0 0" xyz="-0.05004282189881282 -3.3760863741549227e-17 0.033515838063892314"/>
-    <mass value="0.3965131118741336"/>
-    <inertia ixx="0.000347" ixy="-0.0" ixz="-0.0" iyy="0.00096" iyz="-0.0" izz="0.001306"/>
-  </inertial>
-  <visual>
-    <origin rpy="0 0 0" xyz="-0.05 -0.0 -0.001"/>
-    <geometry>
-      <mesh filename="package://maze_robot_v1_description/meshes/base_top_1.stl" scale="0.001 0.001 0.001"/>
-    </geometry>
-    <material name="silver"/>
-  </visual>
-  <collision>
-    <origin rpy="0 0 0" xyz="-0.05 -0.0 -0.001"/>
-    <geometry>
-      <mesh filename="package://maze_robot_v1_description/meshes/base_top_1.stl" scale="0.001 0.001 0.001"/>
-    </geometry>
-  </collision>
-</link>
-<link name="base_top_1">
-  <inertial>
     <origin rpy="0 0 0" xyz="0.04995717810118719 -3.3760863741549227e-17 0.033515838063892314"/>
     <mass value="0.3965131118741336"/>
@@ -181,24 +161,4 @@
     <geometry>
       <mesh filename="package://maze_robot_v1_description/meshes/base_top_1.stl" scale="0.001 0.001 0.001"/>
-    </geometry>
-  </collision>
-</link>
-<link name="main_holder_1">
-  <inertial>
-    <origin rpy="0 0 0" xyz="0.003388479947686096 -0.04900000000000126 0.04655652487203829"/>
-    <mass value="0.769483356673395"/>
-    <inertia ixx="0.001253" ixy="-0.0" ixz="-2.5e-05" iyy="0.000469" iyz="-0.0" izz="0.000955"/>
-  </inertial>
-  <visual>
-    <origin rpy="0 0 0" xyz="-0.0841 -0.049 0.016"/>
-    <geometry>
-      <mesh filename="package://maze_robot_v1_description/meshes/main_holder_1.stl" scale="0.001 0.001 0.001"/>
-    </geometry>
-    <material name="silver"/>
-  </visual>
-  <collision>
-    <origin rpy="0 0 0" xyz="-0.0841 -0.049 0.016"/>
-    <geometry>
-      <mesh filename="package://maze_robot_v1_description/meshes/main_holder_1.stl" scale="0.001 0.001 0.001"/>
     </geometry>
   </collision>

Commit message: update robot description

File: maze_robot_v1_description/urdf/maze_robot_v1.xacro (robot description, xacro)
@@ -84,24 +84,4 @@
   </collision>
 </link>
-<link name="left_wheel_1">
-  <inertial>
-    <origin rpy="0 0 0" xyz="-1.8985381485396353e-15 0.10899999999999999 0.030000000000000006"/>
-    <mass value="0.74505748421744"/>
-    <inertia ixx="0.000253" ixy="-0.0" ixz="-0.0" iyy="0.000409" iyz="-0.0" izz="0.000253"/>
-  </inertial>
-  <visual>
-    <origin rpy="0 0 0" xyz="-0.0 0.0475 0.015"/>
-    <geometry>
-      <mesh filename="package://maze_robot_v1_description/meshes/left_wheel_1.stl" scale="0.001 0.001 0.001"/>
-    </geometry>
-    <material name="silver"/>
-  </visual>
-  <collision>
-    <origin rpy="0 0 0" xyz="-0.0 0.0475 0.015"/>
-    <geometry>
-      <mesh filename="package://maze_robot_v1_description/meshes/left_wheel_1.stl" scale="0.001 0.001 0.001"/>
-    </geometry>
-  </collision>
-</link>
 <link name="support_front_1">
   <inertial>
@@ -146,4 +126,24 @@
 <link name="base_top_1">
   <inertial>
+    <origin rpy="0 0 0" xyz="-0.05004282189881282 -3.3760863741549227e-17 0.033515838063892314"/>
+    <mass value="0.3965131118741336"/>
+    <inertia ixx="0.000347" ixy="-0.0" ixz="-0.0" iyy="0.00096" iyz="-0.0" izz="0.001306"/>
+  </inertial>
+  <visual>
+    <origin rpy="0 0 0" xyz="-0.05 -0.0 -0.001"/>
+    <geometry>
+      <mesh filename="package://maze_robot_v1_description/meshes/base_top_1.stl" scale="0.001 0.001 0.001"/>
+    </geometry>
+    <material name="silver"/>
+  </visual>
+  <collision>
+    <origin rpy="0 0 0" xyz="-0.05 -0.0 -0.001"/>
+    <geometry>
+      <mesh filename="package://maze_robot_v1_description/meshes/base_top_1.stl" scale="0.001 0.001 0.001"/>
+    </geometry>
+  </collision>
+</link>
+<link name="base_top_1">
+  <inertial>
     <origin rpy="0 0 0" xyz="0.04995717810118719 -3.3760863741549227e-17 0.033515838063892314"/>
     <mass value="0.3965131118741336"/>
@@ -166,4 +166,24 @@
 <link name="main_holder_1">
   <inertial>
+    <origin rpy="0 0 0" xyz="0.003388479947686096 -0.04900000000000126 0.04655652487203829"/>
+    <mass value="0.769483356673395"/>
+    <inertia ixx="0.001253" ixy="-0.0" ixz="-2.5e-05" iyy="0.000469" iyz="-0.0" izz="0.000955"/>
+  </inertial>
+  <visual>
+    <origin rpy="0 0 0" xyz="-0.0841 -0.049 0.016"/>
+    <geometry>
+      <mesh filename="package://maze_robot_v1_description/meshes/main_holder_1.stl" scale="0.001 0.001 0.001"/>
+    </geometry>
+    <material name="silver"/>
+  </visual>
+  <collision>
+    <origin rpy="0 0 0" xyz="-0.0841 -0.049 0.016"/>
+    <geometry>
+      <mesh filename="package://maze_robot_v1_description/meshes/main_holder_1.stl" scale="0.001 0.001 0.001"/>
+    </geometry>
+  </collision>
+</link>
+<link name="main_holder_1">
+  <inertial>
     <origin rpy="0 0 0" xyz="0.10658847994768608 -0.04900000000000126 0.04655652487203829"/>
     <mass value="0.769483356673395"/>
@@ -201,4 +221,24 @@
     <geometry>
       <mesh filename="package://maze_robot_v1_description/meshes/iphone_8_1.stl" scale="0.001 0.001 0.001"/>
+    </geometry>
+  </collision>
+</link>
+<link name="left_wheel_1">
+  <inertial>
+    <origin rpy="0 0 0" xyz="-1.856614593209107e-15 0.137 3.469446951953614e-18"/>
+    <mass value="0.7450574842174399"/>
+    <inertia ixx="0.000253" ixy="0.0" ixz="0.0" iyy="0.000409" iyz="-0.0" izz="0.000253"/>
+  </inertial>
+  <visual>
+    <origin rpy="0 0 0" xyz="-0.0 0.0755 -0.015"/>
+    <geometry>
+      <mesh filename="package://maze_robot_v1_description/meshes/left_wheel_1.stl" scale="0.001 0.001 0.001"/>
+    </geometry>
+    <material name="silver"/>
+  </visual>
+  <collision>
+    <origin rpy="0 0 0" xyz="-0.0 0.0755 -0.015"/>
+    <geometry>
+      <mesh filename="package://maze_robot_v1_description/meshes/left_wheel_1.stl" scale="0.001 0.001 0.001"/>
     </geometry>
   </collision>
@@ -220,10 +260,4 @@
   <axis xyz="0.0 1.0 0.0"/>
 </joint>
-<joint name="Rev9" type="continuous">
-  <origin rpy="0 0 0" xyz="0.0 0.0 -0.012"/>
-  <parent link="left_motor_1"/>
-  <child link="left_wheel_1"/>
-  <axis xyz="0.0 1.0 0.0"/>
-</joint>
 <joint name="Rigid10" type="fixed">
   <origin rpy="0 0 0" xyz="0.05 0.0 0.003"/>
@@ -261,3 +295,9 @@
   <child link="iphone_8_1"/>
 </joint>
+<joint name="Rev19" type="continuous">
+  <origin rpy="0 0 0" xyz="0.0 -0.028 0.018"/>
+  <parent link="left_motor_1"/>
+  <child link="left_wheel_1"/>
+  <axis xyz="0.0 1.0 0.0"/>
+</joint>
 </robot>
